File: elec/recepteur 32khz/recepteur 32khz.sch (KiCad schematic (older format))
At the start: 3 parts, among them P11 CONN_7, P4 CONN_6, P5 CONN_6

Commit message: Add some documentation
Other:
- note added: "Beacon 1 - 32.8kHz receiver"
- note added: "Beacon 2 - 32.8kHz receiver"
- note added: "Beacon 3 - 32.8kHz receiver"
- moved on the sheet: P11
Changed lines of the file:
@@
 Connection ~ 3900 2000
 $Sheet
-S 6400 1600 750  400
+S 6700 1500 750  400
 U 551AFB56
 F0 "receiver_32_3-1" 50
 F1 "receiver_32_3-1.sch" 50
-F2 "6V" I L 6400 1750 60
-F3 "GND" I L 6400 1950 60
-F4 "5V" I L 6400 1850 60
-F5 "12V" I L 6400 1650 60
-F6 "Trigger" I R 7150 1800 60
+F2 "6V" I L 6700 1650 60
+F3 "GND" I L 6700 1850 60
+F4 "5V" I L 6700 1750 60
+F5 "12V" I L 6700 1550 60
+F6 "Trigger" I R 7450 1700 60
 $EndSheet
 $Comp
 L recepteur-32khz-rescue:CONN_7 P11
 U 1 1 551B3A29
-P 6800 850
-F 0 "P11" V 6770 850 60  0000 C CNN
-F 1 "CONN_7" V 6870 850 60  0000 C CNN
-F 2 "" H 6800 850 60  0000 C CNN
-F 3 "" H 6800 850 60  0000 C CNN
-	1    6800 850
+P 7100 750
+F 0 "P11" V 7070 750 60  0000 C CNN
+F 1 "CONN_7" V 7170 750 60  0000 C CNN
+F 2 "" H 7100 750 60  0000 C CNN
+F 3 "" H 7100 750 60  0000 C CNN
+	1    7100 750
 	0    -1   -1   0
 $EndComp
 Wire Wire Line
-	6500 1200 5850 1200
+	6800 1100 6150 1100
 Wire Wire Line
-	5850 1200 5850 1650
+	6150 1100 6150 1550
 Wire Wire Line
-	5850 1650 6400 1650
+	6150 1550 6700 1550
 Wire Wire Line
-	6600 1200 6600 1250
+	6900 1100 6900 1150
 Wire Wire Line
-	6600 1250 5900 1250
+	6900 1150 6200 1150
 Wire Wire Line
-	5900 1250 5900 1750
+	6200 1150 6200 1650
 Wire Wire Line
-	5900 1750 6400 1750
+	6200 1650 6700 1650
 Wire Wire Line
-	6700 1200 6700 1300
+	7000 1100 7000 1200
 Wire Wire Line
-	6700 1300 5950 1300
+	7000 1200 6250 1200
 Wire Wire Line
-	5950 1300 5950 1850
+	6250 1200 6250 1750
 Wire Wire Line
-	5950 1850 6400 1850
+	6250 1750 6700 1750
 Wire Wire Line
-	6800 1200 6800 1350
+	7100 1100 7100 1250
 Wire Wire Line
-	6800 1350 6000 1350
+	7100 1250 6300 1250
 Wire Wire Line
-	6000 1350 6000 1950
+	6300 1250 6300 1850
 Wire Wire Line
-	6000 1950 6400 1950
+	6300 1850 6700 1850
 Wire Wire Line
-	7150 1800 7200 1800
+	7450 1700 7500 1700
 Wire Wire Line
-	7200 1800 7200 1500
+	7500 1700 7500 1400
 Wire Wire Line
-	7200 1500 6900 1500
+	7500 1400 7200 1400
 Wire Wire Line
-	6900 1500 6900 1200
+	7200 1400 7200 1100
 $Sheet
-S 6400 2200 750  400
+S 6700 2100 750  400
 U 551C0F76
 F0 "receiver_32_3-2" 50
 F1 "receiver_32_3-2.sch" 50
-F2 "6V" I L 6400 2350 60
-F3 "GND" I L 6400 2550 60
-F4 "5V" I L 6400 2450 60
-F5 "12V" I L 6400 2250 60
-F6 "Trigger" I R 7150 2400 60
+F2 "6V" I L 6700 2250 60
+F3 "GND" I L 6700 2450 60
+F4 "5V" I L 6700 2350 60
+F5 "12V" I L 6700 2150 60
+F6 "Trigger" I R 7450 2300 60
 $EndSheet
 Wire Wire Line
-	7150 2400 7250 2400
+	7450 2300 7550 2300
 Wire Wire Line
-	7250 2400 7250 1450
+	7550 2300 7550 1350
 Wire Wire Line
-	7250 1450 7000 1450
+	7550 1350 7300 1350
 Wire Wire Line
-	7000 1450 7000 1200
+	7300 1350 7300 1100
 Wire Wire Line
-	5850 2250 6400 2250
-Connection ~ 5850 1650
+	6150 2150 6700 2150
+Connection ~ 6150 1550
 Wire Wire Line
-	5900 2350 6400 2350
-Connection ~ 5900 1750
+	6200 2250 6700 2250
+Connection ~ 6200 1650
 Wire Wire Line
-	5950 2450 6400 2450
-Connection ~ 5950 1850
+	6250 2350 6700 2350
+Connection ~ 6250 1750
 Wire Wire Line
-	6000 2550 6400 2550
-Connection ~ 6000 1950
+	6300 2450 6700 2450
+Connection ~ 6300 1850
 $Sheet
-S 6400 2900 750  400
+S 6700 2800 750  400
 U 551C3EAD
 F0 "receiver_32_3-3" 50
 F1 "receiver_32_3-3.sch" 50
-F2 "6V" I L 6400 3050 60
-F3 "GND" I L 6400 3250 60
-F4 "5V" I L 6400 3150 60
-F5 "12V" I L 6400 2950 60
-F6 "Trigger" I R 7150 3100 60
+F2 "6V" I L 6700 2950 60
+F3 "GND" I L 6700 3150 60
+F4 "5V" I L 6700 3050 60
+F5 "12V" I L 6700 2850 60
+F6 "Trigger" I R 7450 3000 60
 $EndSheet
 Wire Wire Line
-	7150 3100 7300 3100
+	7450 3000 7600 3000
 Wire Wire Line
-	7300 3100 7300 1400
+	7600 3000 7600 1300
 Wire Wire Line
-	7300 1400 7100 1400
+	7600 1300 7400 1300
 Wire Wire Line
-	7100 1400 7100 1200
+	7400 1300 7400 1100
 Wire Wire Line
-	6000 3250 6400 3250
-Connection ~ 6000 2550
+	6300 3150 6700 3150
+Connection ~ 6300 2450
 Wire Wire Line
-	5950 3150 6400 3150
-Connection ~ 5950 2450
+	6250 3050 6700 3050
+Connection ~ 6250 2350
 Wire Wire Line
-	5900 3050 6400 3050
-Connection ~ 5900 2350
+	6200 2950 6700 2950
+Connection ~ 6200 2250
 Wire Wire Line
-	5850 2950 6400 2950
-Connection ~ 5850 2250
+	6150 2850 6700 2850
+Connection ~ 6150 2150
 Wire Wire Line
 	1300 1600 1300 2300
@@
 	3900 2000 3900 2700
 Wire Wire Line
-	5850 1650 5850 2250
+	6150 1550 6150 2150
 Wire Wire Line
-	5900 1750 5900 2350
+	6200 1650 6200 2250
 Wire Wire Line
-	5950 1850 5950 2450
+	6250 1750 6250 2350
 Wire Wire Line
-	6000 1950 6000 2550
+	6300 1850 6300 2450
 Wire Wire Line
-	6000 2550 6000 3250
+	6300 2450 6300 3150
 Wire Wire Line
-	5950 2450 5950 3150
+	6250 2350 6250 3050
 Wire Wire Line
-	5900 2350 5900 3050
+	6200 2250 6200 2950
 Wire Wire Line
-	5850 2250 5850 2950
+	6150 2150 6150 2850
+Text Notes 1250 2850 0    50   ~ 0
+Beacon 1 - 32.8kHz receiver
+Text Notes 3700 2950 0    50   ~ 0
+Beacon 2 - 32.8kHz receiver
+Text Notes 6100 3400 0    50   ~ 0
+Beacon 3 - 32.8kHz receiver
+Wire Notes Line
+	1200 2900 1200 750
+Wire Notes Line
+	1200 750  2750 750
+Wire Notes Line
+	2750 750  2750 2900
+Wire Notes Line
+	2750 2900 1200 2900
+Wire Notes Line
+	3650 3000 3650 700
+Wire Notes Line
+	3650 700  5350 700
+Wire Notes Line
+	5350 700  5350 3000
+Wire Notes Line
+	5350 3000 3650 3000
+Wire Notes Line
+	6050 3450 6050 550
+Wire Notes Line
+	6050 550  7800 550
+Wire Notes Line
+	7800 550  7800 3450
+Wire Notes Line
+	7800 3450 6050 3450
 $EndSCHEMATC
